Commit message: Make Gazebo tags optional and minor fixes in colors/inertias

File: talos_description/urdf/arm/arm.urdf.xacro (robot description, xacro)
@@ -147,42 +147,46 @@
                           soft_upper_limit="${0.0 * deg_to_rad - arm_eps}" /> -->
     </joint>
-   <gazebo reference="${name}_${side}_1_link">
-     <mu1>0.9</mu1>
-     <mu2>0.9</mu2>
-     <material>Gazebo/FlatBlack</material>
-   </gazebo>
-   <gazebo reference="${name}_${side}_2_link">
-     <mu1>0.9</mu1>
-     <mu2>0.9</mu2>
-     <material>Gazebo/FlatBlack</material>
-   </gazebo>
-   <gazebo reference="${name}_${side}_3_link">
-     <mu1>0.9</mu1>
-     <mu2>0.9</mu2>
-     <material>Gazebo/FlatBlack</material>
-   </gazebo>
-   <gazebo reference="${name}_${side}_4_link">
-     <mu1>0.9</mu1>
-     <mu2>0.9</mu2>
-     <material>Gazebo/FlatBlack</material>
-   </gazebo>
-   <gazebo reference="${name}_${side}_1_joint">
-      <implicitSpringDamper>1</implicitSpringDamper>
-   </gazebo>
-   <gazebo reference="${name}_${side}_2_joint">
-      <implicitSpringDamper>1</implicitSpringDamper>
-   </gazebo>
-   <gazebo reference="${name}_${side}_3_joint">
-      <implicitSpringDamper>1</implicitSpringDamper>
-   </gazebo>
-   <gazebo reference="${name}_${side}_4_joint">
-      <implicitSpringDamper>1</implicitSpringDamper>
-   </gazebo>
+   <xacro:if value="$(arg enable_gazebo)">
+    <gazebo reference="${name}_${side}_1_link">
+      <mu1>0.9</mu1>
+      <mu2>0.9</mu2>
+      <material>Gazebo/FlatBlack</material>
+    </gazebo>
+    <gazebo reference="${name}_${side}_2_link">
+      <mu1>0.9</mu1>
+      <mu2>0.9</mu2>
+      <material>Gazebo/FlatBlack</material>
+    </gazebo>
+    <gazebo reference="${name}_${side}_3_link">
+      <mu1>0.9</mu1>
+      <mu2>0.9</mu2>
+      <material>Gazebo/FlatBlack</material>
+    </gazebo>
+    <gazebo reference="${name}_${side}_4_link">
+      <mu1>0.9</mu1>
+      <mu2>0.9</mu2>
+      <material>Gazebo/FlatBlack</material>
+    </gazebo>
+    <gazebo reference="${name}_${side}_1_joint">
+        <implicitSpringDamper>1</implicitSpringDamper>
+    </gazebo>
+    <gazebo reference="${name}_${side}_2_joint">
+        <implicitSpringDamper>1</implicitSpringDamper>
+    </gazebo>
+    <gazebo reference="${name}_${side}_3_joint">
+        <implicitSpringDamper>1</implicitSpringDamper>
+    </gazebo>
+    <gazebo reference="${name}_${side}_4_joint">
+        <implicitSpringDamper>1</implicitSpringDamper>
+    </gazebo>
+   </xacro:if>
     <!--************************-->
     <!--        WRIST           -->
     <!--************************-->
      <xacro:talos_wrist name="arm" parent="${name}_${side}_4_link" side="${side}" reflect="${reflect}" />
-    <!-- extensions -->
-    <xacro:include filename="$(find talos_description)/urdf/arm/${side}_arm.transmissions.urdf.xacro" />
+    <xacro:if value="$(arg enable_gazebo)">
+      <!-- extensions -->
+      <xacro:include filename="$(find talos_description)/urdf/arm/${side}_arm.transmissions.urdf.xacro" />
+    </xacro:if>
   </xacro:macro>
 </robot>

File: talos_description/urdf/arm/wrist.urdf.xacro (robot description, xacro)
@@ -112,31 +112,33 @@
                           soft_upper_limit="${40.00000 * deg_to_rad - eps_radians}" /> -->
     </joint>
-    <gazebo reference="${name}_${side}_5_link">
-      <mu1>0.9</mu1>
-      <mu2>0.9</mu2>
-      <material>Gazebo/White</material>
-    </gazebo>
-    <gazebo reference="${name}_${side}_6_link">
-      <mu1>0.9</mu1>
-      <mu2>0.9</mu2>
-      <material>Gazebo/White</material>
-    </gazebo>
-    <gazebo reference="${name}_${side}_7_link">
-      <mu1>0.9</mu1>
-      <mu2>0.9</mu2>
-      <material>Gazebo/FlatBlack</material>
-    </gazebo>
-    <gazebo reference="${name}_${side}_5_joint">
-        <implicitSpringDamper>1</implicitSpringDamper>
-    </gazebo>
-    <gazebo reference="${name}_${side}_6_joint">
-        <implicitSpringDamper>1</implicitSpringDamper>
-    </gazebo>
-    <gazebo reference="${name}_${side}_7_joint">
-        <implicitSpringDamper>1</implicitSpringDamper>
-        <provideFeedback>1</provideFeedback>
-    </gazebo>
-    <!-- extensions -->
-    <xacro:include filename="$(find talos_description)/urdf/arm/${side}_wrist.transmissions.urdf.xacro" />
+    <xacro:if value="$(arg enable_gazebo)">
+      <gazebo reference="${name}_${side}_5_link">
+        <mu1>0.9</mu1>
+        <mu2>0.9</mu2>
+        <material>Gazebo/White</material>
+      </gazebo>
+      <gazebo reference="${name}_${side}_6_link">
+        <mu1>0.9</mu1>
+        <mu2>0.9</mu2>
+        <material>Gazebo/White</material>
+      </gazebo>
+      <gazebo reference="${name}_${side}_7_link">
+        <mu1>0.9</mu1>
+        <mu2>0.9</mu2>
+        <material>Gazebo/FlatBlack</material>
+      </gazebo>
+      <gazebo reference="${name}_${side}_5_joint">
+          <implicitSpringDamper>1</implicitSpringDamper>
+      </gazebo>
+      <gazebo reference="${name}_${side}_6_joint">
+          <implicitSpringDamper>1</implicitSpringDamper>
+      </gazebo>
+      <gazebo reference="${name}_${side}_7_joint">
+          <implicitSpringDamper>1</implicitSpringDamper>
+          <provideFeedback>1</provideFeedback>
+      </gazebo>
+      <!-- extensions -->
+      <xacro:include filename="$(find talos_description)/urdf/arm/${side}_wrist.transmissions.urdf.xacro" />
+    </xacro:if>
   </xacro:macro>
 </robot>

File: talos_description/urdf/gripper/gripper.urdf.xacro (robot description, xacro)
@@ -3,6 +3,8 @@
   <!--File includes-->
   <xacro:include filename="$(find talos_description)/urdf/deg_to_rad.xacro" />
-  <xacro:include filename="$(find talos_description)/urdf/gripper/gripper.transmission.xacro" />
-  <xacro:include filename="$(find talos_description)/urdf/gripper/gripper.gazebo.xacro" />
+  <xacro:if value="$(arg enable_gazebo)">
+    <xacro:include filename="$(find talos_description)/urdf/gripper/gripper.transmission.xacro" />
+    <xacro:include filename="$(find talos_description)/urdf/gripper/gripper.gazebo.xacro" />
+  </xacro:if>
   <xacro:macro name="talos_gripper" params="name parent reflect">
             <link name="${name}_base_link">
@@ -13,5 +15,5 @@
                   <mesh filename="package://talos_description/meshes/gripper/base_link.dae" scale="1 1 1"/>
                 </geometry>
-                <material name="Black"/>
+                <material name="Black" />
               </visual>
               <collision>
@@ -27,5 +29,4 @@
               <origin xyz="0.00000 0.00000 -0.02875"
                       rpy="${0.00000 * deg_to_rad} ${0.00000 * deg_to_rad} ${0.00000 * deg_to_rad}"/>
-              <axis xyz="0 0 0" />
             </joint>
             <link name="${name}_motor_double_link">
@@ -36,5 +37,5 @@
                   <mesh filename="package://talos_description/meshes/gripper/gripper_motor_double.dae" scale="1 1 1"/>
                 </geometry>
-              <material name="Orange"/>
+                <material name="Orange" />
               </visual>
               <collision>
@@ -61,5 +62,5 @@
                   <mesh filename="package://talos_description/meshes/gripper/inner_double.dae" scale="1 1 1"/>
                 </geometry>
-              <material name="Orange"/>
+                <material name="Orange" />
               </visual>
               <collision>
@@ -86,5 +87,5 @@
                   <mesh filename="package://talos_description/meshes/gripper/fingertip.dae" scale="1 1 1"/>
                 </geometry>
-                <material name="Black"/>
+                <material name="Black" />
               </visual>
               <collision>
@@ -111,5 +112,5 @@
                   <mesh filename="package://talos_description/meshes/gripper/fingertip.dae" scale="1 1 1"/>
                 </geometry>
-                <material name="Black"/>
+                <material name="Black" />
               </visual>
               <collision>
@@ -136,5 +137,5 @@
                   <mesh filename="package://talos_description/meshes/gripper/gripper_motor_single.dae" scale="1 1 1"/>
                 </geometry>
-                <material name="Orange"/>
+                <material name="Orange" />
               </visual>
               <collision>
@@ -161,5 +162,5 @@
                   <mesh filename="package://talos_description/meshes/gripper/inner_single.dae" scale="1 1 1"/>
                 </geometry>
-              <material name="Orange"/>
+                <material name="Orange" />
               </visual>
               <collision>
@@ -186,5 +187,5 @@
                   <mesh filename="package://talos_description/meshes/gripper/fingertip.dae" scale="1 1 1"/>
                 </geometry>
-              <material name="Black"/>
+                <material name="Black" />
               </visual>
               <collision>
@@ -204,6 +205,8 @@
               <mimic joint="${name}_joint" multiplier="${-1.0}" offset="0.0" />
             </joint>
-        <xacro:virtual_joints name="${name}" />
-        <xacro:gripper_transmission name="${name}" reduction="1.0" />
+        <xacro:if value="$(arg enable_gazebo)">
+          <xacro:virtual_joints name="${name}" />
+          <xacro:gripper_transmission name="${name}" reduction="1.0" />
+        </xacro:if>
         <!-- virtual mimic joints -->
 <!--         <xacro:gripper_virtual_transmission name="${name}_inner_double" reduction="1.0"/>

File: talos_description/urdf/head/head.urdf.xacro (robot description, xacro)
@@ -51,14 +51,16 @@
                           soft_upper_limit="${45.00000 * deg_to_rad - eps_radians}" /> -->
     </joint>
-    <gazebo reference="${name}_link">
-      <mu1>0.9</mu1>
-      <mu2>0.9</mu2>
-    </gazebo>
-    <gazebo reference="${name}_joint">
-       <implicitSpringDamper>1</implicitSpringDamper>
-    </gazebo>
-    <gazebo reference="${name}_link">
-      <material>Gazebo/FlatBlack</material>
-    </gazebo>
+    <xacro:if value="$(arg enable_gazebo)">
+      <gazebo reference="${name}_link">
+        <mu1>0.9</mu1>
+        <mu2>0.9</mu2>
+      </gazebo>
+      <gazebo reference="${name}_joint">
+        <implicitSpringDamper>1</implicitSpringDamper>
+      </gazebo>
+      <gazebo reference="${name}_link">
+        <material>Gazebo/FlatBlack</material>
+      </gazebo>
+    </xacro:if>
   </xacro:macro>
   <!--************************-->
@@ -95,17 +97,19 @@
                           soft_upper_limit="${75.00000 * deg_to_rad - eps_radians}" /> -->
     </joint>
-    <gazebo reference="${name}_link">
-      <mu1>0.9</mu1>
-      <mu2>0.9</mu2>
-      <material>Gazebo/White</material>
-    </gazebo>
-    <gazebo reference="${name}_joint">
-       <implicitSpringDamper>1</implicitSpringDamper>
-    </gazebo>
+    <xacro:if value="$(arg enable_gazebo)">
+      <gazebo reference="${name}_link">
+        <mu1>0.9</mu1>
+        <mu2>0.9</mu2>
+        <material>Gazebo/White</material>
+      </gazebo>
+      <gazebo reference="${name}_joint">
+        <implicitSpringDamper>1</implicitSpringDamper>
+      </gazebo>
+    </xacro:if>
   </xacro:macro>
-  <xacro:macro name="talos_head" params="name parent disable_gazebo_camera:=false">
+  <xacro:macro name="talos_head" params="name parent">
     <xacro:talos_head_1 name="${name}_1" parent="${parent}" />
     <xacro:talos_head_2 name="${name}_2" parent="${name}_1_link"/>
-    <xacro:orbbec_astra_pro name="rgbd" parent="${name}_2" disable_gazebo="${disable_gazebo_camera}">
+    <xacro:orbbec_astra_pro name="rgbd" parent="${name}_2" enable_gazebo="$(arg enable_gazebo)">
       <!-- Pose of sensor frame wrt to base -->
       <origin xyz="${camera_position_x} ${camera_position_y} ${camera_position_z}" rpy="${camera_orientation_r} ${camera_orientation_p} ${camera_orientation_y}" />
@@ -113,8 +117,10 @@
       <origin xyz="0 0 0" rpy="${-90 * deg_to_rad} 0 ${-90 * deg_to_rad}"/>
     </xacro:orbbec_astra_pro>
-    <xacro:talos_head_differential_transmission name="${name}" number1="1" number2="2"
-                                                act_reduction1="1.0" act_reduction2="1.0"
-                                                jnt_reduction1="1.0" jnt_reduction2="2.0"
-                                                offset_value_1="${head_1_joint_offset}" offset_value_2="${head_2_joint_offset}"/>
+    <xacro:if value="$(arg enable_gazebo)">
+      <xacro:talos_head_differential_transmission name="${name}" number1="1" number2="2"
+                                                  act_reduction1="1.0" act_reduction2="1.0"
+                                                  jnt_reduction1="1.0" jnt_reduction2="2.0"
+                                                  offset_value_1="${head_1_joint_offset}" offset_value_2="${head_2_joint_offset}"/>
+    </xacro:if>
   </xacro:macro>
 </robot>

File: talos_description/urdf/leg/leg.urdf.xacro (robot description, xacro)
@@ -172,78 +172,80 @@
       <dynamics friction="${leg_friction}" damping="${leg_damping}"/>
     </joint>
-    <xacro:talos_leg_simple_transmission side="${prefix}" number="1" reduction="${leg_reduction}" />
-    <xacro:talos_leg_simple_transmission side="${prefix}" number="2" reduction="${leg_reduction}" />
-    <xacro:talos_leg_simple_transmission side="${prefix}" number="3" reduction="${leg_reduction}" />
-    <xacro:talos_leg_simple_transmission side="${prefix}" number="4" reduction="${leg_reduction}" />
-    <xacro:talos_leg_simple_transmission side="${prefix}" number="5" reduction="${leg_reduction}" />
-    <xacro:talos_leg_simple_transmission side="${prefix}" number="6" reduction="${leg_reduction}" />
-   <gazebo reference="leg_${prefix}_1_link">
-     <mu1>0.9</mu1>
-     <mu2>0.9</mu2>
-   </gazebo>
-   <gazebo reference="leg_${prefix}_2_link">
-     <mu1>0.9</mu1>
-     <mu2>0.9</mu2>
-   </gazebo>
-   <gazebo reference="leg_${prefix}_3_link">
-     <mu1>0.9</mu1>
-     <mu2>0.9</mu2>
-   </gazebo>
-   <gazebo reference="leg_${prefix}_4_link">
-     <mu1>0.9</mu1>
-     <mu2>0.9</mu2>
-   </gazebo>
-   <gazebo reference="leg_${prefix}_5_link">
-     <mu1>0.9</mu1>
-     <mu2>0.9</mu2>
-   </gazebo>
-   <!-- contact model for foot surface -->
-   <gazebo reference="leg_${prefix}_6_link">
-    <kp>1000000.0</kp>
-    <kd>100.0</kd>
-    <mu1>1.0</mu1>
-    <mu2>1.0</mu2>
-    <fdir1>1 0 0</fdir1>
-    <maxVel>1.0</maxVel>
-    <minDepth>0.00</minDepth>
-    <implicitSpringDamper>1</implicitSpringDamper>
-   </gazebo>
-   <gazebo reference="leg_${prefix}_1_joint">
+    <xacro:if value="$(arg enable_gazebo)">
+      <xacro:talos_leg_simple_transmission side="${prefix}" number="1" reduction="${leg_reduction}" />
+      <xacro:talos_leg_simple_transmission side="${prefix}" number="2" reduction="${leg_reduction}" />
+      <xacro:talos_leg_simple_transmission side="${prefix}" number="3" reduction="${leg_reduction}" />
+      <xacro:talos_leg_simple_transmission side="${prefix}" number="4" reduction="${leg_reduction}" />
+      <xacro:talos_leg_simple_transmission side="${prefix}" number="5" reduction="${leg_reduction}" />
+      <xacro:talos_leg_simple_transmission side="${prefix}" number="6" reduction="${leg_reduction}" />
+    <gazebo reference="leg_${prefix}_1_link">
+      <mu1>0.9</mu1>
+      <mu2>0.9</mu2>
+    </gazebo>
+    <gazebo reference="leg_${prefix}_2_link">
+      <mu1>0.9</mu1>
+      <mu2>0.9</mu2>
+    </gazebo>
+    <gazebo reference="leg_${prefix}_3_link">
+      <mu1>0.9</mu1>
+      <mu2>0.9</mu2>
+    </gazebo>
+    <gazebo reference="leg_${prefix}_4_link">
+      <mu1>0.9</mu1>
+      <mu2>0.9</mu2>
+    </gazebo>
+    <gazebo reference="leg_${prefix}_5_link">
+      <mu1>0.9</mu1>
+      <mu2>0.9</mu2>
+    </gazebo>
+    <!-- contact model for foot surface -->
+    <gazebo reference="leg_${prefix}_6_link">
+      <kp>1000000.0</kp>
+      <kd>100.0</kd>
+      <mu1>1.0</mu1>
+      <mu2>1.0</mu2>
+      <fdir1>1 0 0</fdir1>
+      <maxVel>1.0</maxVel>
+      <minDepth>0.00</minDepth>
       <implicitSpringDamper>1</implicitSpringDamper>
-   </gazebo>
-   <gazebo reference="leg_${prefix}_2_joint">
+    </gazebo>
+    <gazebo reference="leg_${prefix}_1_joint">
+        <implicitSpringDamper>1</implicitSpringDamper>
+    </gazebo>
+    <gazebo reference="leg_${prefix}_2_joint">
+        <implicitSpringDamper>1</implicitSpringDamper>
+    </gazebo>
+    <gazebo reference="leg_${prefix}_3_joint">
+        <implicitSpringDamper>1</implicitSpringDamper>
+    </gazebo>
+    <gazebo reference="leg_${prefix}_4_joint">
+        <implicitSpringDamper>1</implicitSpringDamper>
+    </gazebo>
+    <gazebo reference="leg_${prefix}_5_joint">
+        <implicitSpringDamper>1</implicitSpringDamper>
+    </gazebo>
+    <gazebo reference="leg_${prefix}_6_joint">
       <implicitSpringDamper>1</implicitSpringDamper>
-   </gazebo>
-   <gazebo reference="leg_${prefix}_3_joint">
-      <implicitSpringDamper>1</implicitSpringDamper>
-   </gazebo>
-   <gazebo reference="leg_${prefix}_4_joint">
-      <implicitSpringDamper>1</implicitSpringDamper>
-   </gazebo>
-   <gazebo reference="leg_${prefix}_5_joint">
-      <implicitSpringDamper>1</implicitSpringDamper>
-   </gazebo>
-   <gazebo reference="leg_${prefix}_6_joint">
-     <implicitSpringDamper>1</implicitSpringDamper>
-     <provideFeedback>1</provideFeedback>
-   </gazebo>
-  <gazebo reference="leg_${prefix}_1_link">
-    <material>Gazebo/FlatBlack</material>
-  </gazebo>
-  <gazebo reference="leg_${prefix}_2_link">
-    <material>Gazebo/FlatBlack</material>
-  </gazebo>
-  <gazebo reference="leg_${prefix}_3_link">
-    <material>Gazebo/FlatBlack</material>
-  </gazebo>
-  <gazebo reference="leg_${prefix}_4_link">
-    <material>Gazebo/FlatBlack</material>
-  </gazebo>
-  <gazebo reference="leg_${prefix}_5_link">
-    <material>Gazebo/White</material>
-  </gazebo>
-  <gazebo reference="leg_${prefix}_6_link">
-    <material>Gazebo/White</material>
-  </gazebo>
+      <provideFeedback>1</provideFeedback>
+    </gazebo>
+    <gazebo reference="leg_${prefix}_1_link">
+      <material>Gazebo/FlatBlack</material>
+    </gazebo>
+    <gazebo reference="leg_${prefix}_2_link">
+      <material>Gazebo/FlatBlack</material>
+    </gazebo>
+    <gazebo reference="leg_${prefix}_3_link">
+      <material>Gazebo/FlatBlack</material>
+    </gazebo>
+    <gazebo reference="leg_${prefix}_4_link">
+      <material>Gazebo/FlatBlack</material>
+    </gazebo>
+    <gazebo reference="leg_${prefix}_5_link">
+      <material>Gazebo/White</material>
+    </gazebo>
+    <gazebo reference="leg_${prefix}_6_link">
+      <material>Gazebo/White</material>
+    </gazebo>
+  </xacro:if>
   </xacro:macro>
 </robot>

File: talos_description/urdf/sensors/ftsensor.urdf.xacro (robot description, xacro)
@@ -43,5 +43,5 @@
           <cylinder radius="${0.05*0.5}" length="0.00975"/>
         </geometry>
-        <material name="FlatBlack" />
+        <material name="Black" />
       </visual>
       <collision>

File: talos_description/urdf/sensors/imu.urdf.xacro (robot description, xacro)
@@ -16,4 +16,5 @@
           <box size="0.01 0.01 0.01"/>
         </geometry>
+        <material name="White"/> <!-- Not sure about this -->
       </visual>
     </link>

File: talos_description/urdf/sensors/orbbec_astra_pro.urdf.xacro (robot description, xacro)
@@ -20,5 +20,5 @@
   <xacro:include filename="$(find talos_description)/urdf/sensors/orbbec_astra_pro.gazebo.xacro" />
   <!-- Macro -->
-  <xacro:macro name="orbbec_astra_pro" params="name parent *origin *optical_origin disable_gazebo:=false">
+  <xacro:macro name="orbbec_astra_pro" params="name parent *origin *optical_origin enable_gazebo:=true">
     <!-- frames in the center of the camera -->
     <joint name="${name}_joint" type="fixed">
@@ -59,5 +59,7 @@
       <child link="${name}_depth_frame"/>
     </joint>
-    <link name="${name}_depth_frame"/>
+    <link name="${name}_depth_frame">
+      <xacro:call macro="${name}_optical_frame_inertial" />
+    </link>
     <joint name="${name}_depth_optical_joint" type="fixed">
       <origin xyz="0 0 0" rpy="${-90.0 * deg_to_rad} 0.0 ${-90.0 * deg_to_rad}" />
@@ -65,5 +67,7 @@
       <child link="${name}_depth_optical_frame"/>
     </joint>
-    <link name="${name}_depth_optical_frame"/>
+    <link name="${name}_depth_optical_frame">
+      <xacro:call macro="${name}_optical_frame_inertial" />
+    </link>
     <!-- frames of the rgb sensor -->
     <joint name="${name}_rgb_joint" type="fixed">
@@ -72,5 +76,7 @@
       <child link="${name}_rgb_frame"/>
     </joint>
-    <link name="${name}_rgb_frame"/>
+    <link name="${name}_rgb_frame">
+      <xacro:call macro="${name}_optical_frame_inertial" />
+    </link>
     <joint name="${name}_rgb_optical_joint" type="fixed">
       <origin xyz="0 0 0" rpy="${-90.0 * deg_to_rad} 0.0 ${-90.0 * deg_to_rad}" />
@@ -78,9 +84,11 @@
       <child link="${name}_rgb_optical_frame"/>
     </joint>
-    <link name="${name}_rgb_optical_frame"/>
-    <xacro:unless value="${disable_gazebo}">
+    <link name="${name}_rgb_optical_frame">
+      <xacro:call macro="${name}_optical_frame_inertial" />
+    </link>
+    <xacro:if value="${enable_gazebo}">
       <!-- extensions -->
       <xacro:orbbec_astra_pro_rgbd_camera_gazebo name="${name}" />
-    </xacro:unless>
+    </xacro:if>
   </xacro:macro>
 </robot>

File: talos_description/urdf/talos_full_common.urdf.xacro (robot description, xacro)
@@ -27,5 +27,5 @@
     <xacro:crane parent="torso_2_link"/>
   </xacro:if>
-  <xacro:talos_head name="head" parent="torso_2_link" disable_gazebo_camera="$(arg disable_gazebo_camera)"/>
+  <xacro:talos_head name="head" parent="torso_2_link" />
   <xacro:talos_arm name="arm" parent="torso_2_link" side="left" reflect="1" />
   <xacro:talos_arm name="arm" parent="torso_2_link" side="right" reflect="-1" />
@@ -38,6 +38,8 @@
   <!-- Macro to have the add-on links specific to each TALOS -->
   <xacro:talos_addons />
-  <!-- Generic simulator_gazebo plugins -->
-  <xacro:include filename="$(find talos_description)/gazebo/gazebo.urdf.xacro" />
+  <xacro:if value="$(arg enable_gazebo)">
+    <!-- Generic simulator_gazebo plugins -->
+    <xacro:include filename="$(find talos_description)/gazebo/gazebo.urdf.xacro" />
+  </xacro:if>
   <!-- Materials for visualization -->
   <xacro:include filename="$(find talos_description)/urdf/materials.urdf.xacro" />
