Commit message: Make Gazebo tags optional and minor fixes in colors/inertias

File: talos_description/urdf/torso/torso.urdf.xacro (robot description, xacro)
@@ -27,4 +27,5 @@
           <mesh filename="package://talos_description/meshes/torso/torso_2.dae" scale="1 1 1"/>
         </geometry>
+        <material name="White" />
       </visual>
       <collision>
@@ -45,4 +46,5 @@
           <mesh filename="package://talos_description/meshes/torso/torso_1.dae" scale="1 1 1"/>
         </geometry>
+        <material name="White" />
       </visual>
       <collision>
@@ -78,4 +80,5 @@
           <mesh filename="package://talos_description/meshes/torso/base_link.dae" scale="1 1 1"/>
         </geometry>
+        <material name="White" />
       </visual>
       <collision>
@@ -103,30 +106,32 @@
         <origin xyz="0.04925 0 0.078" rpy="${180.0*deg_to_rad} 0 ${90.0*deg_to_rad}"/>
     </xacro:talos_imu>
-    <gazebo reference="${name}_1_link">
-        <mu1>0.9</mu1>
-        <mu2>0.9</mu2>
-        <material>Gazebo/White</material>
-    </gazebo>
-    <gazebo reference="${name}_2_link">
-        <mu1>0.9</mu1>
-        <mu2>0.9</mu2>
-        <material>Gazebo/White</material>
-    </gazebo>
-    <gazebo reference="base_link">
-        <mu1>0.9</mu1>
-        <mu2>0.9</mu2>
-        <material>Gazebo/White</material>
-    </gazebo>
-    <gazebo reference="${name}_1_joint">
-        <implicitSpringDamper>1</implicitSpringDamper>
-    </gazebo>
-    <gazebo reference="${name}_2_joint">
-        <implicitSpringDamper>1</implicitSpringDamper>
-        <provideFeedback>1</provideFeedback>
-    </gazebo>
-    <!-- extensions -->
-    <xacro:talos_torso_differential_transmission name="${name}" number1="1" number2="2"
-                                                act_reduction1="1.0" act_reduction2="1.0"
-                                                jnt_reduction1="1.0" jnt_reduction2="1.0" />
+    <xacro:if value="$(arg enable_gazebo)">
+      <gazebo reference="${name}_1_link">
+          <mu1>0.9</mu1>
+          <mu2>0.9</mu2>
+          <material>Gazebo/White</material>
+      </gazebo>
+      <gazebo reference="${name}_2_link">
+          <mu1>0.9</mu1>
+          <mu2>0.9</mu2>
+          <material>Gazebo/White</material>
+      </gazebo>
+      <gazebo reference="base_link">
+          <mu1>0.9</mu1>
+          <mu2>0.9</mu2>
+          <material>Gazebo/White</material>
+      </gazebo>
+      <gazebo reference="${name}_1_joint">
+          <implicitSpringDamper>1</implicitSpringDamper>
+      </gazebo>
+      <gazebo reference="${name}_2_joint">
+          <implicitSpringDamper>1</implicitSpringDamper>
+          <provideFeedback>1</provideFeedback>
+      </gazebo>
+      <!-- extensions -->
+      <xacro:talos_torso_differential_transmission name="${name}" number1="1" number2="2"
+                                                  act_reduction1="1.0" act_reduction2="1.0"
+                                                  jnt_reduction1="1.0" jnt_reduction2="1.0" />
+    </xacro:if>
   </xacro:macro>
 </robot>

File: talos_description_inertial/urdf/inertial.xacro (robot description, xacro)
@@ -347,5 +347,5 @@
     <inertial>
       <mass value="0.01"/>
-      <inertia ixx="0" ixy="0" ixz="0" iyy="0" iyz="0" izz="0" />
+      <inertia ixx="1e-06" ixy="0" ixz="0" iyy="1e-06" iyz="0" izz="1e-06"/>
       <origin rpy="0 0 0" xyz="0 0 0"/>
     </inertial>
@@ -382,5 +382,5 @@
     <inertial>
       <mass value="0.001"/>
-      <inertia ixx="0" ixy="0" ixz="0" iyy="0" iyz="0" izz="0" />
+      <inertia ixx="1e-06" ixy="0" ixz="0" iyy="1e-06" iyz="0" izz="1e-06"/>
       <origin rpy="0 0 0" xyz="0 0 0"/>
     </inertial>
@@ -396,5 +396,5 @@
     <inertial>
       <mass value="0.001"/>
-      <inertia ixx="0" ixy="0" ixz="0" iyy="0" iyz="0" izz="0" />
+      <inertia ixx="1e-06" ixy="0" ixz="0" iyy="1e-06" iyz="0" izz="1e-06"/>
       <origin rpy="0 0 0" xyz="0 0 0"/>
     </inertial>
